File: Pinecone V1/Pinecone V1.kicad_pcb (KiCad board)
At the start: 2 copper layers, 50 x 50 mm, 50 parts, among them J2 USB-C, J3 Left, J4 Right, J5 Right, U1 TLV75533PDRV, U2 74AHCT1G125, U3 W25Q128JVPIQ, U4 USBLC6-2SC6, U5 RP2040, Y1 12Mhz

Commit message: Fixed a Resistor Value Typo
Parts:
- added G***: LOGO, LOGO, B.Cu at (113.0, 75.0)
- moved C5 1.41 mm to (107.4, 72.0)
Routing:
- net GND: track 13.5 -> 172.5 mm, vias 6 -> 30
- net Net-(R6-Pad1): track 0.68 -> 27.6 mm, vias 1 -> 2
- net +3V3: track 128.8 -> 137.9 mm, vias 0 -> 2
- net Net-(U5-RUN): track 73.6 -> 80.1 mm
- net VBUS: track 70.4 -> 71.6 mm
- added copper zone on B.Cu, net GND
- added copper zone on F.Cu, net GND

Commit message: PCB V2
Parts:
- removed C18: 10µF, Capacitor_SMD:C_0603_1608Metric
- removed C19: 0.1µF, Capacitor_SMD:C_0402_1005Metric
- removed D2: SK6812MINI, LED_SMD:LED_SK6812MINI_PLCC4_3.5x3.5mm_P1.75mm
- removed R9: 330Ω, Resistor_SMD:R_0402_1005Metric
- removed U2: 74AHCT1G125, Package_TO_SOT_SMD:SOT-353_SC-70-5
Routing:
- net NeoPixel: track 85.4 -> 0.00 mm, vias 2 -> 0
- net GND: track 172.5 -> 152.1 mm, vias 30 -> 27
- net VBUS: track 71.6 -> 62.9 mm
- net Net-(D2-DIN): track 4.79 -> 0.00 mm
- net Net-(R9-Pad2): track 1.11 -> 0.00 mm
