File: Pinecone V1/Pinecone V1.kicad_sch (KiCad schematic)
At the start: 50 parts, among them J2 USB-C, J3 Left, J4 Right, J5 Right, SW1 BOOT, SW2 RESET, U1 TLV75533PDRV, U2 74AHCT1G125, U3 W25Q128JVPIQ, U4 USBLC6-2SC6, U5 RP2040, Y1 12Mhz

Commit message: Fixed a Resistor Value Typo
Parts:
- R10: value 680kΩ -> 680Ω
Changed lines of the file:
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@@
 			)
 		)
-		(property "Value" "680kΩ"
+		(property "Value" "680Ω"
 			(at 200.66 78.232 0)
 			(show_name no)

Commit message: PCB V2
Parts:
- removed C18: 10µF, Capacitor_SMD:C_0603_1608Metric, symbol Device:C_Small
- removed C19: 0.1µF, Capacitor_SMD:C_0402_1005Metric, symbol Device:C_Small
- removed D2: SK6812MINI, LED_SMD:LED_SK6812MINI_PLCC4_3.5x3.5mm_P1.75mm, symbol LED:SK6812MINI
- removed R9: 330Ω, Resistor_SMD:R_0402_1005Metric, symbol Device:R_Small
- removed U2: 74AHCT1G125, Package_TO_SOT_SMD:SOT-353_SC-70-5, symbol 74xGxx:74AHCT1G125
Connections:
- net NeoPixel: no longer names the net of U5.37 (GPIO25)
Other:
- note removed: "NeoPixel"
- moved on the sheet: J3, J4, J5
